File: numpad/PCB/RGBnumpad/RGBnumpad.kicad_pcb (KiCad board)
At the start: 2 copper layers, 100 x 114.3 mm, 67 parts, among them SW1 Rotary_Encoder_Switch, SW2 SW_PUSH, U1 ProMicro

Commit message: routing
curvyyyy
Parts:
- moved SW2 1.39 mm to (52.7, 138.7)
- moved MX13 1.27 mm to (81.0, 99.7)
- moved MX9 1.27 mm to (81.0, 80.6)
Routing:
- net GND: track 538.4 -> 553.2 mm
- net Net-(D2-Pad2): track 69.7 -> 83.6 mm
- net Net-(D3-Pad2): track 97.8 -> 110.5 mm
- net Net-(D4-Pad2): track 112.6 -> 124.7 mm
- net ENCB: track 49.4 -> 61.2 mm
- net ENCA: track 50.3 -> 60.8 mm
- net Net-(D6-Pad2): track 69.5 -> 77.9 mm
- net ROW5: track 84.9 -> 91.7 mm, vias 0 -> 1
- net Net-(D1-Pad2): track 53.2 -> 58.4 mm
- net Net-(LED18-Pad2): track 29.5 -> 34.4 mm
- net Net-(D5-Pad2): track 47.6 -> 52.2 mm
- net Net-(LED4-Pad2): track 82.9 -> 86.7 mm
- net VCC: track 501.1 -> 504.6 mm
- net COL1: track 128.9 -> 132.2 mm
- net ROW4: track 72.9 -> 75.7 mm
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